File: PCB/cuttingboard.kicad_sch (KiCad schematic)
At the start: 33 parts, among them J1 USB_C_Receptacle_USB2.0_14P, J2 Conn_01x20, J3 Conn_01x20, J4 Conn_01x03, SW1 SW_Push, U1 RP2040, U3 W25Q128JVS, U4 MCP1700x-330xxTT, Y1 12 MHz

Commit message: updated devboard to new thing, added Accelerometer
Parts:
- added C18, C20: 0.1uF, Capacitor_SMD:C_0402_1005Metric, symbol Device:C
- added C19: 2.2nf, Capacitor_SMD:C_0402_1005Metric, symbol Device:C
- added R8, R9: 4.7k, Resistor_SMD:R_0402_1005Metric, symbol Device:R
- added U2: MPU-6050, Sensor_Motion:InvenSense_QFN-24_4x4mm_P0.5mm, symbol Sensor_Motion:MPU-6050
Connections:
- net +3V3: now also C20.2, R8.1, R9.2, U2.13 (VDD), U2.8 (VLOGIC)
- net GND: now also C18.1, C19.1, C20.1, U2.1 (CLKIN), U2.11 (FSYNC), U2.18 (GND), U2.9 (AD0)
- net GPIO4: now also R8.2, U2.24 (SDA)
- net GPIO5: now also R9.1, U2.23 (SCL)
- net GPIO25: now reaches U1.37 (GPIO25)
- net GPIO25: now also U2.12 (INT)
- new net: C18.2, U2.10 (REGOUT)
- new net: C19.2, U2.20 (CPOUT)
- no-connect marks 1 -> 2
Other:
- note added: "BUILT-IN ACCELEROMETER"
- moved on the sheet: R3, R4, U1

Commit message: added firmware and updated pcb files
Parts:
- added D1: LED, LED_SMD:LED_0805_2012Metric_Pad1.15x1.40mm_HandSolder, symbol Device:LED
- added R10: 1K, Resistor_SMD:R_0402_1005Metric, symbol Device:R
Connections:
- net GND: now also D1.1 (K)
- net GPIO0: now also R10.2
- new net: D1.2 (A), R10.1
Other:
- note added: "LED"
